Commit message: fixed Rviz visualization in WSL

File: master_ws/src/meshes_robot_description/urdf/robot_arm.urdf.xacro (robot description, xacro)
@@ -4,41 +4,41 @@
 <xacro:include filename="$(find meshes_robot_description)/urdf/gazebo_essentials_arm.xacro" />
   <link name="world"/>
-  <link name="arm_base">
-    <inertial>
-      <origin
-        xyz="7.7128E-09 -0.063005 -3.01969999961422E-08"
-        rpy="0 0 0" />
-      <mass
-        value="1.6004" />
-      <inertia
-        ixx="0.00552196561445819"
-        ixy="7.9550614501301E-10"
-        ixz="-1.34378458924839E-09"
-        iyy="0.00352397447953875"
-        iyz="-1.10071809773382E-08"
-        izz="0.00553739792746489" />
-    </inertial>
-    <visual>
-      <origin
-        xyz="0 0 0"
-        rpy="0 0 0" />
-      <geometry>
-        <mesh filename="package://meshes_robot_description/meshes/arm_base.stl" />
-      </geometry>
-      <material
-        name="">
-        <color
-          rgba="0.79216 0.81961 0.93333 1" />
-      </material>
-    </visual>
-    <collision>
-      <origin
-        xyz="0 0 0"
-        rpy="0 0 0" />
-      <geometry>
-        <mesh filename="package://meshes_robot_description/meshes/arm_base.stl" />
-      </geometry>
-    </collision>
-</link>
+<link name="arm_base">
+  <inertial>
+    <origin
+      xyz="7.7128E-09 -0.063005 -3.01969999961422E-08"
+      rpy="0 0 0" />
+    <mass
+      value="1.6004" />
+    <inertia
+      ixx="0.00552196561445819"
+      ixy="7.9550614501301E-10"
+      ixz="-1.34378458924839E-09"
+      iyy="0.00352397447953875"
+      iyz="-1.10071809773382E-08"
+      izz="0.00553739792746489" />
+  </inertial>
+  <visual>
+    <origin
+      xyz="0 0 0"
+      rpy="0 0 0" />
+    <geometry>
+      <mesh filename="package://meshes_robot_description/meshes/arm_base.stl" />
+    </geometry>
+    <material
+      name="">
+      <color
+        rgba="0.79216 0.81961 0.93333 1" />
+    </material>
+  </visual>
+  <collision>
+    <origin
+      xyz="0 0 0"
+      rpy="0 0 0" />
+    <geometry>
+      <mesh filename="package://meshes_robot_description/meshes/arm_base.stl" />
+    </geometry>
+  </collision>
+  </link>
 <link
     name="bicep">
@@ -194,5 +194,5 @@
   </link>
 <!--######################################################################-->
-<!--<xacro:arm_joint prefix="arm_base" parent="world" child="arm_base" originxyz="0.0 0.0 0.1" originrpy="0 0 0"/>-->
+<!-- <xacro:arm_joint prefix="arm_base" parent="world" child="arm_base" originxyz="0.0 0.0 0.1" originrpy="0 0 0"/> -->
 <joint name="arm_base_joint" type="continuous">
   <axis xyz="0 0 1"/>
@@ -202,7 +202,7 @@
 </joint>
 <xacro:arm_joint prefix="shoulder" parent="arm_base" child="bicep" originxyz="-0.05166 0.0 0.20271" originrpy="0 0 1.5708"/>
-<xacro:arm_joint prefix="bottom_wrist" parent="bicep" child="bottom_wrist" originxyz="0.0 -0.05194 0.269" originrpy="0 0 0"/>
-<!--<xacro:arm_joint prefix="elbow" parent="bottom_wrist" child="elbow" originxyz="0.0 0 0.13522" originrpy="0 0 0"/>-->
-<joint name="elbow_joint" type="continuous">
+<xacro:arm_joint prefix="elbow" parent="bicep" child="bottom_wrist" originxyz="0.0 -0.05194 0.269" originrpy="0 0 0"/>
+<!-- <xacro:arm_joint prefix="elbow" parent="bottom_wrist" child="elbow" originxyz="0.0 0 0.13522" originrpy="0 0 0"/> -->
+<joint name="bottom_wrist" type="continuous">
   <axis xyz="0 0 1"/>
   <parent link="bottom_wrist"/>
