Commit message: attaching robotiq gripper to UR5

File: master_ws/src/custom_robot_description/urdf/6_axis_robot.urdf (robot description, URDF)
Before this commit: robot custom_robot, 1 links, 1 joints
Links:
- removed link tool_0
- added link world
Joints:
- removed joint link_6__tool_0
- added joint fixed: type fixed, parent world, child base_link

File: master_ws/src/custom_robot_description/urdf/custom_gripper.xacro (robot description, xacro)
@@ -5,5 +5,5 @@
     <xacro:macro name="custom_gripper" params="parent origin_xyz">
         <xacro:cobot_link_cylinder name="gripper_connector" origin_xyz="0.0 0.0 0.015" origin_rpy="0.0 0.0 0.0"
-                                    radius="0.04" length="0.03" />
+                                    radius="0.04" length="0.03" mass="0.5" i_xx="0.0002375" i_xy="0" i_xz="0" i_yy="0.0002375" i_yz="0" i_zz="0.00006666666667"/>
         <joint name="{parent}_gripper_connector" type="fixed">
             <parent link="${parent}"/>
@@ -12,5 +12,5 @@
         </joint>
         <xacro:cobot_link_box name="finger_support" origin_xyz="0.0 0.005 0.005" origin_rpy="0.0 0.0 0.0"
-                                    size="0.120 0.01 0.01"/>
+                                    size="0.120 0.01 0.01" mass="0.25" i_xx="0.0003" i_xy="0" i_xz="0" i_yy="0" i_yz="0" i_zz="0.0003"/>
         <joint name="finger_support_gripper_connector" type="fixed">
             <parent link="gripper_connector"/>
@@ -19,7 +19,7 @@
         </joint>
         <xacro:cobot_link_box name="finger_right" origin_xyz="0.0 0.0 0.04" origin_rpy="0.0 0.0 0.0"
-                                    size="0.01 0.01 0.08"/>
+                                    size="0.01 0.01 0.08" mass="0.2" i_xx="0.00042667" i_xy="0" i_xz="0" i_yy="0" i_yz="0" i_zz="0.00042667"/>
         <xacro:cobot_link_box name="finger_left" origin_xyz="0.0 0.0 0.04" origin_rpy="0.0 0.0 0.0"
-                                    size="0.01 0.01 0.08"/>
+                                    size="0.01 0.01 0.08" mass="0.2" i_xx="0.00042667" i_xy="0" i_xz="0" i_yy="0" i_yz="0" i_zz="0.00042667"/>
         <joint name="finger_right_joint" type="prismatic">
             <parent link="finger_support"/>
@@ -39,4 +39,10 @@
             <mimic joint="finger_right_joint" multiplier="-1.0" offset="0" />
         </joint>
+        <xacro:transmission name="trans_finger_right_joint"
+                        joint_name="finger_right_joint"
+                        actuator_name = "motor_finger_right_joint"/>
+        <xacro:transmission name="trans_finger_left_joint"
+                        joint_name="finger_left_joint"
+                        actuator_name = "motor_finger_left_joint"/>
     </xacro:macro>
 </robot>

File: master_ws/src/custom_robot_description/urdf/link_joint.xacro (robot description, xacro)
@@ -1,6 +1,11 @@
 <?xml version = "1.0"?>
 <robot xmlns:xacro="http://www.ros.org/wiki/xacro">
-    <xacro:macro name="cobot_link_cylinder" params="name origin_xyz origin_rpy radius length">
+    <xacro:macro name="cobot_link_cylinder" params="name origin_xyz origin_rpy radius length mass i_xx i_xy i_xz i_yy i_yz i_zz">
         <link name="${name}">
+            <inertial>
+                <origin xyz="${origin_xyz}" rpy="${origin_rpy}"/>
+                <mass value="${mass}"/>
+                <inertia ixx="${i_xx}" ixy="${i_xy}" ixz="${i_xz}" iyy="${i_yy}" iyz="${i_yz}" izz="${i_zz}"/>
+            </inertial>
             <visual>
                 <geometry>
@@ -17,6 +22,11 @@
         </link>
     </xacro:macro>
-    <xacro:macro name="cobot_link_box" params="name origin_xyz origin_rpy size">
+    <xacro:macro name="cobot_link_box" params="name origin_xyz origin_rpy size mass i_xx i_xy i_xz i_yy i_yz i_zz">
         <link name="${name}">
+            <inertial>
+                <origin xyz="${origin_xyz}" rpy="${origin_rpy}"/>
+                <mass value="${mass}"/>
+                <inertia ixx="${i_xx}" ixy="${i_xy}" ixz="${i_xz}" iyy="${i_yy}" iyz="${i_yz}" izz="${i_zz}"/>
+            </inertial>
             <visual>
                 <geometry>
@@ -42,3 +52,15 @@
         </joint>
     </xacro:macro>
+    <xacro:macro name="transmission" params="name joint_name actuator_name">
+        <transmission name="${name}" >
+            <type>transmission_interface/SimpleTransmission</type>
+            <joint name= "${joint_name}" >
+                <hardwareInterface>hardware_interface/EffortJointInterface</hardwareInterface>
+            </joint>
+            <actuator name= "${actuator_name}" >
+                <hardwareInterface>hardware_interface/EffortJointInterface</hardwareInterface>
+                <mechanicalReduction>1</mechanicalReduction>
+            </actuator>
+        </transmission>
+    </xacro:macro>
 </robot>

Commit message: PID controllers for custom robot is tuned

File: master_ws/src/custom_robot_description/urdf/6_axis_robot.urdf (robot description, URDF)
Before this commit: robot custom_robot, 1 links, 1 joints
Links:
- added link tool_0
Joints:
- added joint link_6__tool_0: type fixed, parent link_6, child tool_0, origin xyz=0.0 0.0 0.02 rpy=0.0 0.0 0.0

File: master_ws/src/custom_robot_description/urdf/6_axis_robot_gazebo.xacro (robot description, xacro)
@@ -4,4 +4,5 @@
         <plugin name="gazebo_ros_control" filename="libgazebo_ros_control.so">
             <robotNamespace>/cobot</robotNamespace>
+            <!-- <robotSimType>gazebo_ros_control/DefaultRobotHWSim</robotSimType> -->
         </plugin>
     </gazebo>
@@ -40,3 +41,22 @@
         <material>Gazebo/Blue</material>
     </gazebo>
+    <!-- ros control plugin to mimic finger behavior-->
+    <xacro:macro name="mimic_joint_plugin_gazebo" params="parent_joint mimic_joint has_pid:=false multiplier:=-1.0 offset:=0 sensitiveness:=0.0 max_effort:=200 robot_namespace:='/cobot'">
+        <gazebo>
+            <plugin name="${mimic_joint}_mimic_joint_plugin" filename="libroboticsgroup_gazebo_mimic_joint_plugin.so">
+                <joint>${parent_joint}</joint>
+                <mimicJoint>${mimic_joint}</mimicJoint>
+                <xacro:if value="${has_pid}">
+                    <hasPID />
+                </xacro:if>
+                <multiplier>${multiplier}</multiplier>
+                <offset>${offset}</offset>
+                <sensitiveness>${sensitiveness}</sensitiveness>
+                <maxEffort>${max_effort}</maxEffort>
+                <xacro:unless value="${robot_namespace == '/cobot'}">
+                    <robotNamespace>($robot_namespace)</robotNamespace>
+                </xacro:unless>
+            </plugin>
+        </gazebo>
+    </xacro:macro>
 </robot>

File: master_ws/src/custom_robot_description/urdf/custom_gripper.xacro (robot description, xacro)
@@ -19,8 +19,35 @@
         </joint>
         <xacro:cobot_link_box name="finger_right" origin_xyz="0.0 0.0 0.04" origin_rpy="0.0 0.0 0.0"
-                                    size="0.01 0.01 0.08" mass="0.2" i_xx="0.00042667" i_xy="0" i_xz="0" i_yy="0" i_yz="0" i_zz="0.00042667"/>
+                                    size="0.01 0.01 0.08" mass="0.2" i_xx="0.00042667" i_xy="0" i_xz="0"
+                                    i_yy="0.00042667" i_yz="0" i_zz="0.0000083"/>
         <xacro:cobot_link_box name="finger_left" origin_xyz="0.0 0.0 0.04" origin_rpy="0.0 0.0 0.0"
-                                    size="0.01 0.01 0.08" mass="0.2" i_xx="0.00042667" i_xy="0" i_xz="0" i_yy="0" i_yz="0" i_zz="0.00042667"/>
+                                    size="0.01 0.01 0.08" mass="0.2" i_xx="0.00042667" i_xy="0" i_xz="0"
+                                    i_yy="0.00042667" i_yz="0" i_zz="0.0000083"/>
         <joint name="finger_right_joint" type="prismatic">
+            <parent link="finger_support"/>
+            <child link="finger_right"/>
+            <axis xyz="1 0 0"/>
+            <limit lower="0" upper="0.044" velocity="0.5" effort="200"/>
+            <origin xyz="-0.05 0.0 0.011" rpy="0 0 0"/>
+            <dynamics damping="1" friction="2"/>
+        </joint>
+        <xacro:transmission name="trans_finger_right_joint"
+                        joint_name="finger_right_joint"
+                        actuator_name="motor_finger_right_joint" />
+        <joint name="finger_left_joint" type="prismatic">
+            <parent link="finger_support"/>
+            <child link="finger_left"/>
+            <axis xyz="1 0 0"/>
+            <limit lower="-0.044" upper="0" velocity="0.5" effort="200"/>
+            <origin xyz="0.05 0.0 0.011" rpy="0 0 0"/>
+            <dynamics damping="1" friction="2"/>
+            <mimic joint="finger_right_joint" multiplier="-1.0" offset="0" />
+        </joint>
+        <xacro:transmission name="trans_finger_left_joint"
+                        joint_name="finger_left_joint"
+                        actuator_name="motor_finger_left_joint" />
+        <xacro:mimic_joint_plugin_gazebo  parent_joint="finger_right_joint" mimic_joint="finger_left_joint"
+                                            has_pid="false" multiplier="-1.0" max_effort="200" />
+        <!-- <joint name="finger_right_joint" type="prismatic">
             <parent link="finger_support"/>
             <child link="finger_right"/>
@@ -45,4 +72,6 @@
                         joint_name="finger_left_joint"
                         actuator_name = "motor_finger_left_joint"/>
+        <xacro:mimic_joint_plugin_gazebo  parent_joint="finger_right_joint" mimic_joint="finger_left_joint"
+                                            has_pid="false" multiplier="-1.0" max_effort="200" /> -->
     </xacro:macro>
 </robot>
