Commit message: path planning and collision avoidance

File: master_ws/src/custom_robot_description/urdf/6_axis_robot.urdf.xacro (robot description, xacro)
@@ -13,4 +13,5 @@
         <parent link="world"/>
         <child link="base_link"/>
+        <origin xyz="0 0.0 0.8" rpy="0 0 0"/>
     </joint>
     <!-- Create Link 1 using xacro-->
@@ -220,4 +221,11 @@
         <child link="tool_0"/>
         <origin xyz="0.0 0.0 0.02" rpy="0.0 0.0 0.0"/>
+    </joint>
+    <link name="picking_point">
+    </link>
+    <joint name="tool_0_picking_point" type="fixed">
+        <parent link="tool_0"/>
+        <child link="picking_point"/>
+        <origin xyz="0.0 0.0 0.08" rpy="0.0 0.0 0.0"/>
     </joint>
     <xacro:custom_gripper parent="tool_0" origin_xyz="0.0 0.0 0.0"/>

File: master_ws/src/custom_robot_description/urdf/6_axis_robot_gazebo.xacro (robot description, xacro)
@@ -60,3 +60,23 @@
         </gazebo>
     </xacro:macro>
+    <!-- gazebo grasp fix plugin to grasp the object without sliding-->
+    <gazebo>
+        <plugin name="gazebo_grasp_fix" filename="libgazebo_grasp_fix.so">
+            <arm>
+                <arm_name>custom_gripper</arm_name>
+                <!-- The link which the finger joints are attached -->
+                <palm_link> link_6  </palm_link>
+                <gripper_link> finger_right </gripper_link>
+                <gripper_link> finger_left </gripper_link>
+                <gripper_link> ... </gripper_link>
+            </arm>
+            <forces_angle_tolerance>100</forces_angle_tolerance>
+            <update_rate>4</update_rate>
+            <grip_count_threshold>4</grip_count_threshold>
+            <max_grip_count>8</max_grip_count>
+            <release_tolerance>0.005</release_tolerance>
+            <disable_collisions_on_attach>false</disable_collisions_on_attach>
+            <contact_topic>__default_topic__</contact_topic>
+        </plugin>
+    </gazebo>
 </robot>
